File: EAGLE/ChessPCB.brd (EAGLE design)
At the start: 94.2 x 76.3 mm, 22 parts

Commit message: PCB Updates
Parts:
- added R4: (no value), rcl:0204/7
- added X12: (no value), ME507:2POL254
- moved R1 2.54 mm to (61.0, 7.62)
- moved R2 2.54 mm to (61.0, 3.81)
- moved X4 2.54 mm to (48.3, 8.89)
- moved FERBEAD 1.27 mm to (25.4, 72.4)
Connections:
- new net N$32: R4.1, X12.2
- net GND: now also X12.1
- net N$24: now also R4.2
Routing:
- net N$24: track 73.7 -> 100.3 mm
- net N$23: track 207.7 -> 217.8 mm
- net N$32: track 0.00 -> 5.21 mm
- net N$27: track 36.2 -> 40.7 mm
- net N$30: track 133.1 -> 129.8 mm
- net N$21: track 83.8 -> 86.4 mm
- net N$19: track 71.2 -> 73.7 mm
- net N$20: track 4.48 -> 5.75 mm
Other:
- board size 94.2 x 76.3 mm -> 91.7 x 76.3 mm
- board text added: "5V"
- board text added: "ADAFRUIT BSS138 LVL SHIFT"
- board text added: "AO1"
- board text added: "AO2"
- board text added: "BO1"
- board text added: "BO2"
- board text added: "CLW"
- board text added: "CO1"
- board text added: "CO2"
- board text added: "DONE"
- board text added: "EA+"
- board text added: "EA-"
- board text added: "EA5"
- board text added: "EB+"
- board text added: "EB-"
- board text added: "EB5"
- board text added: "GND"
- board text added: "LED"
- board text added: "LM1"
- board text added: "LM2"
- board text added: "LV2"
- board text added: "POLOLU TB6612FNG MTR DRV"
- board text added: "RST"
- board text added: "STOP"
- board text added: "Sigma Phi Delta - Chess Robot Project Corey Agena, Andrew Hudak, Ivan Nieto, Jeffrey Wexler, Vishesh Pithadiya, Edgar Rojas"
- board text added: "VCC"
- board text added: "VMOT"
