File: EAGLE/ChessPCB.sch (EAGLE design)
At the start: 22 parts

Commit message: PCB Edits
Parts:
- X7: device ME507:SCREWTERM_3P_254 -> ME507:SCREWTERM_2P_254
Connections:
- net GND: now also X7-1.1; no longer X7-2.1
- net N$17: now also LV.2; no longer LV.3
- net N$22: now also X7-2.1; no longer X7-3.1
- net N$8: now also LV.3; no longer LV.2
Other:
- moved on the sheet: X7-2
Changed lines of the file:
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@@
 <part name="R3" library="rcl" library_urn="urn:adsk.eagle:library:334" deviceset="R-EU_" device="0204/7" package3d_urn="urn:adsk.eagle:package:23498/2"/>
 <part name="GND16" library="SparkFun-PowerSymbols" library_urn="urn:adsk.eagle:library:530" deviceset="GND" device=""/>
-<part name="X7" library="ME507" deviceset="SCREWTERM_3P" device="_254"/>
+<part name="X7" library="ME507" deviceset="SCREWTERM_2P" device="_254"/>
 </parts>
 <sheets>
@@
 <attribute name="VALUE" x="-0.254" y="88.9" size="1.778" layer="96" rot="R270" align="top-center"/>
 </instance>
-<instance part="X7" gate="-2" x="7.62" y="91.44" smashed="yes" rot="R90">
+<instance part="X7" gate="-1" x="7.62" y="91.44" smashed="yes" rot="R90">
 <attribute name="NAME" x="8.255" y="94.996" size="1.778" layer="95" rot="R90"/>
 </instance>
-<instance part="X7" gate="-3" x="12.7" y="91.44" smashed="yes" rot="R90">
+<instance part="X7" gate="-2" x="12.7" y="91.44" smashed="yes" rot="R90">
 <attribute name="NAME" x="13.335" y="94.996" size="1.778" layer="95" rot="R90"/>
 <attribute name="VALUE" x="16.002" y="90.424" size="1.778" layer="96" rot="R90"/>
@@
 </segment>
 <segment>
-<pinref part="X7" gate="-2" pin="1"/>
 <pinref part="GND16" gate="1" pin="GND"/>
 <wire x1="7.62" y1="88.9" x2="2.54" y2="88.9" width="0.1524" layer="91"/>
+<pinref part="X7" gate="-1" pin="1"/>
 </segment>
 </net>
@@
 <wire x1="25.4" y1="48.26" x2="40.64" y2="48.26" width="0.1524" layer="91"/>
 <wire x1="25.4" y1="20.32" x2="-20.32" y2="20.32" width="0.1524" layer="91"/>
-<wire x1="-20.32" y1="20.32" x2="-20.32" y2="7.62" width="0.1524" layer="91"/>
-<pinref part="LV" gate="G$1" pin="2"/>
-<wire x1="-20.32" y1="7.62" x2="-17.78" y2="7.62" width="0.1524" layer="91"/>
+<wire x1="-20.32" y1="20.32" x2="-20.32" y2="5.08" width="0.1524" layer="91"/>
+<pinref part="LV" gate="G$1" pin="3"/>
+<wire x1="-20.32" y1="5.08" x2="-17.78" y2="5.08" width="0.1524" layer="91"/>
 </segment>
 </net>
@@
 <wire x1="22.86" y1="50.8" x2="40.64" y2="50.8" width="0.1524" layer="91"/>
 <wire x1="22.86" y1="22.86" x2="-22.86" y2="22.86" width="0.1524" layer="91"/>
-<wire x1="-22.86" y1="22.86" x2="-22.86" y2="5.08" width="0.1524" layer="91"/>
-<pinref part="LV" gate="G$1" pin="3"/>
-<wire x1="-22.86" y1="5.08" x2="-17.78" y2="5.08" width="0.1524" layer="91"/>
+<wire x1="-22.86" y1="22.86" x2="-22.86" y2="7.62" width="0.1524" layer="91"/>
+<pinref part="LV" gate="G$1" pin="2"/>
+<wire x1="-22.86" y1="7.62" x2="-17.78" y2="7.62" width="0.1524" layer="91"/>
 </segment>
 </net>
@@
 <segment>
 <pinref part="R3" gate="G$1" pin="1"/>
-<pinref part="X7" gate="-3" pin="1"/>
 <wire x1="17.78" y1="88.9" x2="12.7" y2="88.9" width="0.1524" layer="91"/>
-</segment>
-</net>
+<pinref part="X7" gate="-2" pin="1"/>
+</segment>
+</net>

Commit message: PCB Updates
Parts:
- added R4: (no value), rcl:R-EU_0204/7
- added X12: (no value), ME507:SCREWTERM_2P_254
Connections:
- new net N$32: R4.1, X12-2.1
- net GND: now also X12-1.1
- net N$24: now also R4.2
Changed lines of the file:
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@@
 <part name="GND16" library="SparkFun-PowerSymbols" library_urn="urn:adsk.eagle:library:530" deviceset="GND" device=""/>
 <part name="X7" library="ME507" deviceset="SCREWTERM_2P" device="_254"/>
+<part name="R4" library="rcl" library_urn="urn:adsk.eagle:library:334" deviceset="R-EU_" device="0204/7" package3d_urn="urn:adsk.eagle:package:23498/2"/>
+<part name="GND25" library="SparkFun-PowerSymbols" library_urn="urn:adsk.eagle:library:530" deviceset="GND" device=""/>
+<part name="X12" library="ME507" deviceset="SCREWTERM_2P" device="_254"/>
 </parts>
 <sheets>
@@
 <attribute name="NAME" x="13.335" y="94.996" size="1.778" layer="95" rot="R90"/>
 <attribute name="VALUE" x="16.002" y="90.424" size="1.778" layer="96" rot="R90"/>
+</instance>
+<instance part="R4" gate="G$1" x="83.82" y="7.62" smashed="yes" rot="R90">
+<attribute name="NAME" x="82.3214" y="3.81" size="1.778" layer="95" rot="R90"/>
+<attribute name="VALUE" x="87.122" y="3.81" size="1.778" layer="96" rot="R90"/>
+</instance>
+<instance part="GND25" gate="1" x="83.82" y="-12.7" smashed="yes">
+<attribute name="VALUE" x="83.82" y="-12.954" size="1.778" layer="96" align="top-center"/>
+</instance>
+<instance part="X12" gate="-1" x="81.28" y="-5.08" smashed="yes" rot="R180">
+<attribute name="NAME" x="77.724" y="-4.445" size="1.778" layer="95" rot="R180"/>
+</instance>
+<instance part="X12" gate="-2" x="81.28" y="0" smashed="yes" rot="R180">
+<attribute name="NAME" x="77.724" y="0.635" size="1.778" layer="95" rot="R180"/>
+<attribute name="VALUE" x="82.296" y="3.302" size="1.778" layer="96" rot="R180"/>
 </instance>
 </instances>
@@
 <wire x1="7.62" y1="88.9" x2="2.54" y2="88.9" width="0.1524" layer="91"/>
 <pinref part="X7" gate="-1" pin="1"/>
+</segment>
+<segment>
+<pinref part="GND25" gate="1" pin="GND"/>
+<wire x1="83.82" y1="-5.08" x2="83.82" y2="-10.16" width="0.1524" layer="91"/>
+<pinref part="X12" gate="-1" pin="1"/>
 </segment>
 </net>
@@
 <pinref part="X4" gate="-2" pin="1"/>
 <pinref part="X4" gate="-4" pin="1"/>
-<wire x1="149.86" y1="12.7" x2="38.1" y2="12.7" width="0.1524" layer="91"/>
+<wire x1="149.86" y1="12.7" x2="83.82" y2="12.7" width="0.1524" layer="91"/>
 <pinref part="HV" gate="G$1" pin="6"/>
+<wire x1="83.82" y1="12.7" x2="38.1" y2="12.7" width="0.1524" layer="91"/>
 <wire x1="7.62" y1="10.16" x2="38.1" y2="10.16" width="0.1524" layer="91"/>
 <junction x="38.1" y="10.16"/>
+<pinref part="R4" gate="G$1" pin="2"/>
+<junction x="83.82" y="12.7"/>
 </segment>
 </net>
@@
 </segment>
 </net>
+<net name="N$32" class="0">
+<segment>
+<pinref part="R4" gate="G$1" pin="1"/>
+<wire x1="83.82" y1="2.54" x2="83.82" y2="0" width="0.1524" layer="91"/>
+<pinref part="X12" gate="-2" pin="1"/>
+</segment>
+</net>
 </nets>
 </sheet>
 </sheets>
+<errors>
+</errors>
 </schematic>
 </drawing>
